File: foxglove/power_supplies.sch (KiCad schematic (older format))
At the start: 13 parts

Commit message: Added iCE40-HX8K-CT256 to schematic, began signal routing.
Parts:
- J6: renamed from J?; symbol Connector:Conn_01x02_Female -> Connector_Generic:Conn_01x02
- gave numbers to parts that had none: 12
Other:
- note added: "add LDO"
Changed lines of the file:
@@
 DAC4
 $Comp
-L gsg-symbols:MC4558CPT U?
+L gsg-symbols:MC4558CPT U20
 U 1 1 5C96A74B
 P 2600 1800
-F 0 "U?" H 2600 2265 50  0000 C CNN
+F 0 "U20" H 2600 2265 50  0000 C CNN
 F 1 "MC4558CPT" H 2600 2174 50  0000 C CNN
 F 2 "" H 2600 1900 50  0001 C CNN
@@
 	2200 1950 2200 2000
 $Comp
-L power:GND #PWR?
+L power:GND #PWR0179
 U 1 1 5C96A9C8
 P 2200 2000
-F 0 "#PWR?" H 2200 1750 50  0001 C CNN
+F 0 "#PWR0179" H 2200 1750 50  0001 C CNN
 F 1 "GND" H 2205 1827 50  0000 C CNN
 F 2 "" H 2200 2000 50  0001 C CNN
@@
 $EndComp
 $Comp
-L Device:C C?
+L Device:C C6
 U 1 1 5C96AA35
 P 3000 1450
-F 0 "C?" H 3115 1496 50  0000 L CNN
+F 0 "C6" H 3115 1496 50  0000 L CNN
 F 1 "0.1uF" H 3115 1405 50  0000 L CNN
 F 2 "" H 3038 1300 50  0001 C CNN
@@
 Connection ~ 3000 1650
 $Comp
-L power:+5V #PWR?
+L power:+5V #PWR0180
 U 1 1 5C96AC55
 P 3050 1650
-F 0 "#PWR?" H 3050 1500 50  0001 C CNN
+F 0 "#PWR0180" H 3050 1500 50  0001 C CNN
 F 1 "+5V" V 3065 1778 50  0000 L CNN
 F 2 "" H 3050 1650 50  0001 C CNN
@@
 $EndComp
 $Comp
-L power:GND #PWR?
+L power:GND #PWR0181
 U 1 1 5C96AC70
 P 3000 1250
-F 0 "#PWR?" H 3000 1000 50  0001 C CNN
+F 0 "#PWR0181" H 3000 1000 50  0001 C CNN
 F 1 "GND" H 3005 1077 50  0000 C CNN
 F 2 "" H 3000 1250 50  0001 C CNN
@@
 	2950 1800 2950 1850
 $Comp
-L gsg-symbols:MC4558CPT U?
+L gsg-symbols:MC4558CPT U21
 U 1 1 5C96C1A9
 P 2600 3200
-F 0 "U?" H 2600 3665 50  0000 C CNN
+F 0 "U21" H 2600 3665 50  0000 C CNN
 F 1 "MC4558CPT" H 2600 3574 50  0000 C CNN
 F 2 "" H 2600 3300 50  0001 C CNN
@@
 	2200 3350 2200 3400
 $Comp
-L power:GND #PWR?
+L power:GND #PWR0182
 U 1 1 5C96C1B2
 P 2200 3400
-F 0 "#PWR?" H 2200 3150 50  0001 C CNN
+F 0 "#PWR0182" H 2200 3150 50  0001 C CNN
 F 1 "GND" H 2205 3227 50  0000 C CNN
 F 2 "" H 2200 3400 50  0001 C CNN
@@
 $EndComp
 $Comp
-L Device:C C?
+L Device:C C7
 U 1 1 5C96C1B8
 P 3000 2850
-F 0 "C?" H 3115 2896 50  0000 L CNN
+F 0 "C7" H 3115 2896 50  0000 L CNN
 F 1 "0.1uF" H 3115 2805 50  0000 L CNN
 F 2 "" H 3038 2700 50  0001 C CNN
@@
 Connection ~ 3000 3050
 $Comp
-L power:+5V #PWR?
+L power:+5V #PWR0183
 U 1 1 5C96C1C3
 P 3050 3050
-F 0 "#PWR?" H 3050 2900 50  0001 C CNN
+F 0 "#PWR0183" H 3050 2900 50  0001 C CNN
 F 1 "+5V" V 3065 3178 50  0000 L CNN
 F 2 "" H 3050 3050 50  0001 C CNN
@@
 $EndComp
 $Comp
-L power:GND #PWR?
+L power:GND #PWR0184
 U 1 1 5C96C1C9
 P 3000 2650
-F 0 "#PWR?" H 3000 2400 50  0001 C CNN
+F 0 "#PWR0184" H 3000 2400 50  0001 C CNN
 F 1 "GND" H 3005 2477 50  0000 C CNN
 F 2 "" H 3000 2650 50  0001 C CNN
@@
 	2950 3200 2950 3250
 $Comp
-L gsg-symbols:DAC084S085 U?
+L gsg-symbols:DAC084S085 U22
 U 1 1 5CA11A45
 P 4100 2400
-F 0 "U?" H 4100 2825 50  0000 C CNN
+F 0 "U22" H 4100 2825 50  0000 C CNN
 F 1 "DAC084S085" H 4100 2734 50  0000 C CNN
 F 2 "" H 4000 2500 50  0001 C CNN
@@
 $EndComp
 $Comp
-L power:+5V #PWR?
+L power:+5V #PWR0185
 U 1 1 5CA11DF8
 P 3650 2150
-F 0 "#PWR?" H 3650 2000 50  0001 C CNN
+F 0 "#PWR0185" H 3650 2000 50  0001 C CNN
 F 1 "+5V" V 3665 2278 50  0000 L CNN
 F 2 "" H 3650 2150 50  0001 C CNN
@@
 SSEL
 $Comp
-L Device:R R?
+L Device:R R24
 U 1 1 5CA148C6
 P 4650 2100
-F 0 "R?" H 4720 2146 50  0000 L CNN
+F 0 "R24" H 4720 2146 50  0000 L CNN
 F 1 "10k" H 4720 2055 50  0000 L CNN
 F 2 "" V 4580 2100 50  0001 C CNN
@@
 	4650 1950 4650 1900
 $Comp
-L power:+5V #PWR?
+L power:+5V #PWR0186
 U 1 1 5CA1736F
 P 4650 1900
-F 0 "#PWR?" H 4650 1750 50  0001 C CNN
+F 0 "#PWR0186" H 4650 1750 50  0001 C CNN
 F 1 "+5V" V 4665 2028 50  0000 L CNN
 F 2 "" H 4650 1900 50  0001 C CNN
@@
 $EndComp
 $Comp
-L power:+5V #PWR?
+L power:+5V #PWR0187
 U 1 1 5CA173C2
 P 4550 2500
-F 0 "#PWR?" H 4550 2350 50  0001 C CNN
+F 0 "#PWR0187" H 4550 2350 50  0001 C CNN
 F 1 "+5V" V 4565 2628 50  0000 L CNN
 F 2 "" H 4550 2500 50  0001 C CNN
@@
 	4500 2500 4550 2500
 $Comp
-L power:GND #PWR?
+L power:GND #PWR0188
 U 1 1 5CA19E9F
 P 4550 2600
-F 0 "#PWR?" H 4550 2350 50  0001 C CNN
+F 0 "#PWR0188" H 4550 2350 50  0001 C CNN
 F 1 "GND" V 4555 2472 50  0000 R CNN
 F 2 "" H 4550 2600 50  0001 C CNN
@@
 	1900 2400 1900 3250
 $Comp
-L Connector:Conn_01x02_Female J?
+L Connector_Generic:Conn_01x02 J6
 U 1 1 5CA47169
 P 1400 2100
-F 0 "J?" H 1294 1775 50  0000 C CNN
+F 0 "J6" H 1294 1775 50  0000 C CNN
 F 1 "Conn_01x02_Female" H 1294 1866 50  0000 C CNN
 F 2 "" H 1400 2100 50  0001 C CNN
@@
 	1650 2100 1650 2150
 $Comp
-L power:GND #PWR?
+L power:GND #PWR0189
 U 1 1 5CA4A02E
 P 1650 2150
-F 0 "#PWR?" H 1650 1900 50  0001 C CNN
+F 0 "#PWR0189" H 1650 1900 50  0001 C CNN
 F 1 "GND" H 1655 1977 50  0000 C CNN
 F 2 "" H 1650 2150 50  0001 C CNN
@@
 optional external \nsupply input
 $Comp
-L gsg-symbols:MIC94310 U?
+L gsg-symbols:MIC94310 U23
 U 1 1 5CA9D75B
 P 7550 2600
-F 0 "U?" H 7550 2550 60  0000 C CNN
+F 0 "U23" H 7550 2550 60  0000 C CNN
 F 1 "MIC94310" H 7550 2650 60  0000 C CNN
 F 2 "" H 7550 2600 60  0001 C CNN
@@
 $EndComp
 $Comp
-L Device:C C?
+L Device:C C9
 U 1 1 5CA9D762
 P 7650 3450
-F 0 "C?" H 7675 3550 50  0000 L CNN
+F 0 "C9" H 7675 3550 50  0000 L CNN
 F 1 "10uF" H 7675 3350 50  0000 L CNN
 F 2 "" H 7688 3300 50  0001 C CNN
@@
 $EndComp
 $Comp
-L Device:C C?
+L Device:C C8
 U 1 1 5CA9D769
 P 7400 1800
-F 0 "C?" H 7425 1900 50  0000 L CNN
+F 0 "C8" H 7425 1900 50  0000 L CNN
 F 1 "0.47uF" H 7425 1700 50  0000 L CNN
 F 2 "" H 7438 1650 50  0001 C CNN
@@
 	7550 2000 7550 1800
 $Comp
-L power:VCC #PWR?
+L power:VCC #PWR0190
 U 1 1 5CA9D771
 P 7200 1800
-F 0 "#PWR?" H 7200 1650 50  0001 C CNN
+F 0 "#PWR0190" H 7200 1650 50  0001 C CNN
 F 1 "VCC" H 7200 1950 50  0000 C CNN
 F 2 "" H 7200 1800 50  0001 C CNN
@@
 	7250 2000 7350 2000
 $Comp
-L power:GND #PWR?
+L power:GND #PWR0191
 U 1 1 5CA9D778
 P 7600 1800
-F 0 "#PWR?" H 7600 1550 50  0001 C CNN
+F 0 "#PWR0191" H 7600 1550 50  0001 C CNN
 F 1 "GND" H 7600 1650 50  0000 C CNN
 F 2 "" H 7600 1800 50  0001 C CNN
@@
 	7550 1800 7600 1800
 $Comp
-L power:VCC #PWR?
+L power:VCC #PWR0192
 U 1 1 5CA9D77F
 P 7850 2000
-F 0 "#PWR?" H 7850 1850 50  0001 C CNN
+F 0 "#PWR0192" H 7850 1850 50  0001 C CNN
 F 1 "VCC" H 7850 2150 50  0000 C CNN
 F 2 "" H 7850 2000 50  0001 C CNN
@@
 	7750 2000 7850 2000
 $Comp
-L power:GND #PWR?
+L power:GND #PWR0193
 U 1 1 5CA9D786
 P 7650 3650
-F 0 "#PWR?" H 7650 3400 50  0001 C CNN
+F 0 "#PWR0193" H 7650 3400 50  0001 C CNN
 F 1 "GND" H 7650 3500 50  0000 C CNN
 F 2 "" H 7650 3650 50  0001 C CNN
@@
 $EndComp
 $Comp
-L gsg-symbols:MIC94310 U?
+L gsg-symbols:MIC94310 U24
 U 1 1 5CA9D78C
 P 8350 2600
-F 0 "U?" H 8350 2550 60  0000 C CNN
+F 0 "U24" H 8350 2550 60  0000 C CNN
 F 1 "MIC94310" H 8350 2650 60  0000 C CNN
 F 2 "" H 8350 2600 60  0001 C CNN
@@
 $EndComp
 $Comp
-L Device:C C?
+L Device:C C11
 U 1 1 5CA9D793
 P 8450 3450
-F 0 "C?" H 8475 3550 50  0000 L CNN
+F 0 "C11" H 8475 3550 50  0000 L CNN
 F 1 "10uF" H 8475 3350 50  0000 L CNN
 F 2 "" H 8488 3300 50  0001 C CNN
@@
 $EndComp
 $Comp
-L Device:C C?
+L Device:C C10
 U 1 1 5CA9D79A
 P 8200 1800
-F 0 "C?" H 8225 1900 50  0000 L CNN
+F 0 "C10" H 8225 1900 50  0000 L CNN
 F 1 "0.47uF" H 8225 1700 50  0000 L CNN
 F 2 "" H 8238 1650 50  0001 C CNN
@@
 	8350 2000 8350 1800
 $Comp
-L power:VCC #PWR?
+L power:VCC #PWR0194
 U 1 1 5CA9D7A2
 P 8000 1800
-F 0 "#PWR?" H 8000 1650 50  0001 C CNN
+F 0 "#PWR0194" H 8000 1650 50  0001 C CNN
 F 1 "VCC" H 8000 1950 50  0000 C CNN
 F 2 "" H 8000 1800 50  0001 C CNN
@@
 	8050 2000 8150 2000
 $Comp
-L power:GND #PWR?
+L power:GND #PWR0195
 U 1 1 5CA9D7A9
 P 8400 1800
-F 0 "#PWR?" H 8400 1550 50  0001 C CNN
+F 0 "#PWR0195" H 8400 1550 50  0001 C CNN
 F 1 "GND" H 8400 1650 50  0000 C CNN
 F 2 "" H 8400 1800 50  0001 C CNN
@@
 	8350 1800 8400 1800
 $Comp
-L power:VCC #PWR?
+L power:VCC #PWR0196
 U 1 1 5CA9D7B0
 P 8650 2000
-F 0 "#PWR?" H 8650 1850 50  0001 C CNN
+F 0 "#PWR0196" H 8650 1850 50  0001 C CNN
 F 1 "VCC" H 8650 2150 50  0000 C CNN
 F 2 "" H 8650 2000 50  0001 C CNN
@@
 	8550 2000 8650 2000
 $Comp
-L power:GND #PWR?
+L power:GND #PWR0197
 U 1 1 5CA9D7B7
 P 8450 3650
-F 0 "#PWR?" H 8450 3400 50  0001 C CNN
+F 0 "#PWR0197" H 8450 3400 50  0001 C CNN
 F 1 "GND" H 8450 3500 50  0000 C CNN
 F 2 "" H 8450 3650 50  0001 C CNN
@@
 Connection ~ 8350 1800
 $Comp
-L power:+1V2 #PWR?
+L power:+1V2 #PWR0198
 U 1 1 5CA9D7C9
 P 7600 3300
-F 0 "#PWR?" H 7600 3150 50  0001 C CNN
+F 0 "#PWR0198" H 7600 3150 50  0001 C CNN
 F 1 "+1V2" V 7615 3428 50  0000 L CNN
 F 2 "" H 7600 3300 50  0001 C CNN
@@
 Connection ~ 8450 3300
 $Comp
-L power:+2V5 #PWR?
+L power:+2V5 #PWR0199
 U 1 1 5CA9D7D4
 P 8400 3300
-F 0 "#PWR?" H 8400 3150 50  0001 C CNN
+F 0 "#PWR0199" H 8400 3150 50  0001 C CNN
 F 1 "+2V5" V 8415 3428 50  0000 L CNN
 F 2 "" H 8400 3300 50  0001 C CNN
@@
 	0    -1   -1   0
 $EndComp
+Text Notes 1450 3350 0    50   ~ 0
+add LDO
 $EndSCHEMATC
