File: bankA_mux.sch (KiCad schematic (older format))
At the start: 7 parts, among them U10 SHIFTER, U9 74HC4051

Commit message: Changed bank A footprint and rearranged silkscreen
Changed lines of the file:
@@
 AR Path="/5D1A4680/5CF3E254" Ref="U21"  Part="1"
 AR Path="/5D1A4696/5CF3E254" Ref="U23"  Part="1"
-F 0 "U21" H 4100 3428 50  0000 C CNN
+F 0 "U23" H 4100 3428 50  0000 C CNN
 F 1 "74HC4051" H 4100 3337 50  0000 C CNN
 F 2 "Package_TO_SOT_SMD:SOT-763-1" H 4050 2350 50  0001 C CNN
@@
 AR Path="/5D1A4680/5CF3E25C" Ref="#PWR0180"  Part="1"
 AR Path="/5D1A4696/5CF3E25C" Ref="#PWR0186"  Part="1"
-F 0 "#PWR0180" H 4100 2100 50  0001 C CNN
+F 0 "#PWR0186" H 4100 2100 50  0001 C CNN
 F 1 "+5V" V 4115 2378 50  0000 L CNN
 F 2 "" H 4100 2250 50  0001 C CNN
@@
 AR Path="/5D1A4680/5CF3E263" Ref="#PWR0181"  Part="1"
 AR Path="/5D1A4696/5CF3E263" Ref="#PWR0187"  Part="1"
-F 0 "#PWR0181" H 4100 3150 50  0001 C CNN
+F 0 "#PWR0187" H 4100 3150 50  0001 C CNN
 F 1 "GND" H 4105 3227 50  0000 C CNN
 F 2 "" H 4100 3400 50  0001 C CNN
@@
 AR Path="/5D1A4680/5CF3E282" Ref="#PWR0182"  Part="1"
 AR Path="/5D1A4696/5CF3E282" Ref="#PWR0188"  Part="1"
-F 0 "#PWR0182" H 4500 1800 50  0001 C CNN
+F 0 "#PWR0188" H 4500 1800 50  0001 C CNN
 F 1 "GND" H 4505 1877 50  0000 C CNN
 F 2 "" H 4500 2050 50  0001 C CNN
@@
 AR Path="/5D1A4680/5CF3E28C" Ref="U22"  Part="1"
 AR Path="/5D1A4696/5CF3E28C" Ref="U24"  Part="1"
-F 0 "U22" H 4100 4350 60  0000 C CNN
+F 0 "U24" H 4100 4350 60  0000 C CNN
 F 1 "SHIFTER" H 4100 3950 60  0000 C CNN
 F 2 "gsg-modules:SOT363" H 4100 4150 60  0001 C CNN
@@
 AR Path="/5D1A4680/5CF3E293" Ref="#PWR0183"  Part="1"
 AR Path="/5D1A4696/5CF3E293" Ref="#PWR0189"  Part="1"
-F 0 "#PWR0183" H 4500 3900 50  0001 C CNN
+F 0 "#PWR0189" H 4500 3900 50  0001 C CNN
 F 1 "GND" H 4500 4000 50  0000 C CNN
 F 2 "" H 4500 4150 60  0000 C CNN
@@
 AR Path="/5D1A4680/5CF3E2A6" Ref="R35"  Part="1"
 AR Path="/5D1A4696/5CF3E2A6" Ref="R38"  Part="1"
-F 0 "R35" V 3780 3250 50  0000 C CNN
+F 0 "R38" V 3780 3250 50  0000 C CNN
 F 1 "10k" V 3700 3250 50  0000 C CNN
 F 2 "gsg-modules:0402" V 3630 3250 50  0001 C CNN
@@
 AR Path="/5D1A4680/5CF3E2B2" Ref="#PWR0184"  Part="1"
 AR Path="/5D1A4696/5CF3E2B2" Ref="#PWR0190"  Part="1"
-F 0 "#PWR0184" H 3700 3300 50  0001 C CNN
+F 0 "#PWR0190" H 3700 3300 50  0001 C CNN
 F 1 "+5V" V 3715 3578 50  0000 L CNN
 F 2 "" H 3700 3450 50  0001 C CNN
@@
 AR Path="/5D1A4680/5CF3E2B8" Ref="#PWR0185"  Part="1"
 AR Path="/5D1A4696/5CF3E2B8" Ref="#PWR0191"  Part="1"
-F 0 "#PWR0185" H 4500 4100 50  0001 C CNN
+F 0 "#PWR0191" H 4500 4100 50  0001 C CNN
 F 1 "VCC" V 4517 4378 50  0000 L CNN
 F 2 "" H 4500 4250 50  0001 C CNN
@@
 AR Path="/5D190D22/5CB0C423" Ref="R51"  Part="1"
 AR Path="/5D1A466A/5CB0C423" Ref="R53"  Part="1"
-F 0 "R54" V 2700 3700 50  0000 C CNN
+F 0 "R55" V 2700 3700 50  0000 C CNN
 F 1 "100" V 2800 3700 50  0000 C CNN
 F 2 "gsg-modules:0402" V 2730 3700 50  0001 C CNN
@@
 AR Path="/5D1A4680/5CDC112C" Ref="R47"  Part="1"
 AR Path="/5D1A4696/5CDC112C" Ref="R62"  Part="1"
-F 0 "R47" V 4830 2250 50  0000 C CNN
+F 0 "R62" V 4830 2250 50  0000 C CNN
 F 1 "10k" V 4750 2250 50  0000 C CNN
 F 2 "gsg-modules:0402" V 4680 2250 50  0001 C CNN
@@
 AR Path="/5D1A4680/5CDC1279" Ref="R46"  Part="1"
 AR Path="/5D1A4696/5CDC1279" Ref="R61"  Part="1"
-F 0 "R46" V 4580 2250 50  0000 C CNN
+F 0 "R61" V 4580 2250 50  0000 C CNN
 F 1 "10k" V 4500 2250 50  0000 C CNN
 F 2 "gsg-modules:0402" V 4430 2250 50  0001 C CNN
@@
 AR Path="/5D1A4680/5D112AA5" Ref="C42"  Part="1"
 AR Path="/5D1A4696/5D112AA5" Ref="C43"  Part="1"
-F 0 "C42" V 3052 3350 50  0000 C CNN
+F 0 "C43" V 3052 3350 50  0000 C CNN
 F 1 "0.1uF" V 2961 3350 50  0000 C CNN
 F 2 "gsg-modules:0402" H 2838 3200 50  0001 C CNN

Commit message: Added silkscreen tables for banks and completed BOM data
Parts:
- R17, R24, R25: Description (none) -> RES 10K OHM 5% 1/16W 0402; Manufacturer (none) -> Stackpole Electronics Inc; Part Number (none) -> RMCF0402JT10K0
Connections:
- net +5V: now also R17.2; no longer R17.1
- net ~E~: now also R17.1; no longer R17.2
Changed lines of the file:
@@
 $Descr A4 11693 8268
 encoding utf-8
-Sheet 5 17
+Sheet 2 17
 Title ""
 Date ""
@@
 AR Path="/5D1A4680/5CF3E254" Ref="U21"  Part="1"
 AR Path="/5D1A4696/5CF3E254" Ref="U23"  Part="1"
-F 0 "U23" H 4100 3428 50  0000 C CNN
+F 0 "U9" H 4100 3428 50  0000 C CNN
 F 1 "74HC4051" H 4100 3337 50  0000 C CNN
 F 2 "Package_TO_SOT_SMD:SOT-763-1" H 4050 2350 50  0001 C CNN
@@
 AR Path="/5D1A4680/5CF3E28C" Ref="U22"  Part="1"
 AR Path="/5D1A4696/5CF3E28C" Ref="U24"  Part="1"
-F 0 "U24" H 4100 4350 60  0000 C CNN
+F 0 "U10" H 4100 4350 60  0000 C CNN
 F 1 "SHIFTER" H 4100 3950 60  0000 C CNN
 F 2 "gsg-modules:SOT363" H 4100 4150 60  0001 C CNN
@@
 Wire Wire Line
 	4450 4150 4500 4150
-$Comp
-L Device:R R?
-U 1 1 5CF3E2A6
-P 3700 3250
-AR Path="/5CF3E2A6" Ref="R?"  Part="1"
-AR Path="/5C7E37E4/5CF37D46/5CF3E2A6" Ref="R?"  Part="1"
-AR Path="/5CF421CD/5CF3E2A6" Ref="R17"  Part="1"
-AR Path="/5D17D622/5CF3E2A6" Ref="R20"  Part="1"
-AR Path="/5D190D0C/5CF3E2A6" Ref="R23"  Part="1"
-AR Path="/5D190D22/5CF3E2A6" Ref="R26"  Part="1"
-AR Path="/5D1A4654/5CF3E2A6" Ref="R29"  Part="1"
-AR Path="/5D1A466A/5CF3E2A6" Ref="R32"  Part="1"
-AR Path="/5D1A4680/5CF3E2A6" Ref="R35"  Part="1"
-AR Path="/5D1A4696/5CF3E2A6" Ref="R38"  Part="1"
-F 0 "R38" V 3780 3250 50  0000 C CNN
-F 1 "10k" V 3700 3250 50  0000 C CNN
-F 2 "gsg-modules:0402" V 3630 3250 50  0001 C CNN
-F 3 "" H 3700 3250 50  0001 C CNN
-	1    3700 3250
-	-1   0    0    1
-$EndComp
 Wire Wire Line
 	3700 3400 3700 3450
@@
 AR Path="/5D190D22/5CB0C423" Ref="R51"  Part="1"
 AR Path="/5D1A466A/5CB0C423" Ref="R53"  Part="1"
-F 0 "R55" V 2700 3700 50  0000 C CNN
+F 0 "R48" V 2700 3700 50  0000 C CNN
 F 1 "100" V 2800 3700 50  0000 C CNN
 F 2 "gsg-modules:0402" V 2730 3700 50  0001 C CNN
@@
 AR Path="/5D1A4680/5CDC112C" Ref="R47"  Part="1"
 AR Path="/5D1A4696/5CDC112C" Ref="R62"  Part="1"
-F 0 "R62" V 4830 2250 50  0000 C CNN
+F 0 "R25" V 4830 2250 50  0000 C CNN
 F 1 "10k" V 4750 2250 50  0000 C CNN
 F 2 "gsg-modules:0402" V 4680 2250 50  0001 C CNN
 F 3 "" H 4750 2250 50  0001 C CNN
+F 4 "Stackpole Electronics Inc" H 4750 2250 50  0001 C CNN "Manufacturer"
+F 5 "RMCF0402JT10K0" H 4750 2250 50  0001 C CNN "Part Number"
+F 6 "RES 10K OHM 5% 1/16W 0402" H 4750 2250 50  0001 C CNN "Description"
 	1    4750 2250
-	1    0    0    -1
-$EndComp
-$Comp
-L Device:R R?
-U 1 1 5CDC1279
-P 4500 2250
-AR Path="/5CDC1279" Ref="R?"  Part="1"
-AR Path="/5C7E37E4/5CF37D46/5CDC1279" Ref="R?"  Part="1"
-AR Path="/5CF421CD/5CDC1279" Ref="R24"  Part="1"
-AR Path="/5D17D622/5CDC1279" Ref="R27"  Part="1"
-AR Path="/5D190D0C/5CDC1279" Ref="R30"  Part="1"
-AR Path="/5D190D22/5CDC1279" Ref="R33"  Part="1"
-AR Path="/5D1A4654/5CDC1279" Ref="R36"  Part="1"
-AR Path="/5D1A466A/5CDC1279" Ref="R39"  Part="1"
-AR Path="/5D1A4680/5CDC1279" Ref="R46"  Part="1"
-AR Path="/5D1A4696/5CDC1279" Ref="R61"  Part="1"
-F 0 "R61" V 4580 2250 50  0000 C CNN
-F 1 "10k" V 4500 2250 50  0000 C CNN
-F 2 "gsg-modules:0402" V 4430 2250 50  0001 C CNN
-F 3 "" H 4500 2250 50  0001 C CNN
-	1    4500 2250
 	1    0    0    -1
 $EndComp
@@
 AR Path="/5D1A4680/5D112AA5" Ref="C42"  Part="1"
 AR Path="/5D1A4696/5D112AA5" Ref="C43"  Part="1"
-F 0 "C43" V 3052 3350 50  0000 C CNN
+F 0 "C20" V 3052 3350 50  0000 C CNN
 F 1 "0.1uF" V 2961 3350 50  0000 C CNN
 F 2 "gsg-modules:0402" H 2838 3200 50  0001 C CNN
@@
 	2950 3350 2950 3700
 Connection ~ 2950 3700
+$Comp
+L Device:R R?
+U 1 1 5D2823C8
+P 4500 2250
+AR Path="/5D2823C8" Ref="R?"  Part="1"
+AR Path="/5C7E37E4/5CF37D46/5D2823C8" Ref="R?"  Part="1"
+AR Path="/5CF421CD/5D2823C8" Ref="R24"  Part="1"
+AR Path="/5D17D622/5D2823C8" Ref="R27"  Part="1"
+AR Path="/5D190D0C/5D2823C8" Ref="R30"  Part="1"
+AR Path="/5D190D22/5D2823C8" Ref="R33"  Part="1"
+AR Path="/5D1A4654/5D2823C8" Ref="R36"  Part="1"
+AR Path="/5D1A466A/5D2823C8" Ref="R39"  Part="1"
+AR Path="/5D1A4680/5D2823C8" Ref="R46"  Part="1"
+AR Path="/5D1A4696/5D2823C8" Ref="R61"  Part="1"
+F 0 "R24" V 4580 2250 50  0000 C CNN
+F 1 "10k" V 4500 2250 50  0000 C CNN
+F 2 "gsg-modules:0402" V 4430 2250 50  0001 C CNN
+F 3 "" H 4500 2250 50  0001 C CNN
+F 4 "Stackpole Electronics Inc" H 4500 2250 50  0001 C CNN "Manufacturer"
+F 5 "RMCF0402JT10K0" H 4500 2250 50  0001 C CNN "Part Number"
+F 6 "RES 10K OHM 5% 1/16W 0402" H 4500 2250 50  0001 C CNN "Description"
+	1    4500 2250
+	1    0    0    -1
+$EndComp
+$Comp
+L Device:R R?
+U 1 1 5D2825B7
+P 3700 3250
+AR Path="/5D2825B7" Ref="R?"  Part="1"
+AR Path="/5C7E37E4/5CF37D46/5D2825B7" Ref="R?"  Part="1"
+AR Path="/5CF421CD/5D2825B7" Ref="R17"  Part="1"
+AR Path="/5D17D622/5D2825B7" Ref="R20"  Part="1"
+AR Path="/5D190D0C/5D2825B7" Ref="R23"  Part="1"
+AR Path="/5D190D22/5D2825B7" Ref="R26"  Part="1"
+AR Path="/5D1A4654/5D2825B7" Ref="R29"  Part="1"
+AR Path="/5D1A466A/5D2825B7" Ref="R32"  Part="1"
+AR Path="/5D1A4680/5D2825B7" Ref="R35"  Part="1"
+AR Path="/5D1A4696/5D2825B7" Ref="R38"  Part="1"
+F 0 "R17" V 3780 3250 50  0000 C CNN
+F 1 "10k" V 3700 3250 50  0000 C CNN
+F 2 "gsg-modules:0402" V 3630 3250 50  0001 C CNN
+F 3 "" H 3700 3250 50  0001 C CNN
+F 4 "Stackpole Electronics Inc" H 3700 3250 50  0001 C CNN "Manufacturer"
+F 5 "RMCF0402JT10K0" H 3700 3250 50  0001 C CNN "Part Number"
+F 6 "RES 10K OHM 5% 1/16W 0402" H 3700 3250 50  0001 C CNN "Description"
+	1    3700 3250
+	1    0    0    -1
+$EndComp
 $EndSCHEMATC
