File: foxglove.sch (KiCad schematic (older format))
At the start: 92 parts, among them IC1 LFE5U-12F-6BG256C, J1 NEIGHBOR1, J2 NEIGHBOR2, J3 Conn_02x05_Odd_Even, J4 Conn_02x05_Odd_Even, J5 Conn_01x02_Female, J6 Conn_02x03_Odd_Even, J7 BONUS_ROW, U1 LM393, U2 ADP225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

Commit message: Changed headers for bank A and B, combined ADC voltage divider / pull-ups
Parts:
- removed J4: Conn_02x05_Odd_Even, gsg-modules:HEADER-2x5, symbol Connector_Generic:Conn_02x05_Odd_Even
- removed R10: 10k, gsg-modules:0402, symbol Device:R
- added J?: Conn_02x10_Odd_Even, Connector_PinHeader_2.54mm:PinHeader_2x10_P2.54mm_Vertical, symbol Connector_Generic:Conn_02x10_Odd_Even
- J3: footprint gsg-modules:HEADER-2x5 -> gsg-modules:2X5-SHROUDED; Description CONN HEADER R/A 10POS 2.54MM -> Conn Shrouded Header F 10 POS 2.54mm Solder ST Thru-Hole; Manufacturer Samtec Inc. -> SparkFun Electronics; Part Number TSW-105-22-T-D-RA -> PRT-08506
Connections:
- net B2 is gone; now on net B2_P: IC1.G1 (PL20A)
- net +5V: now also R45.1, U4.5 (VCC); no longer R45.2
- net A1: now also J3.3 (Pin_3); no longer J3.1 (Pin_1)
- net A1_shift: now also IC1.P13 (PR41A)
- net A2: now also J3.4 (Pin_4); no longer J3.2 (Pin_2)
- net A2_shift: now also IC1.N16 (PR32A)
- net A3: now also J3.5 (Pin_5); no longer J3.3 (Pin_3)
- net A3_shift: now also IC1.L16 (PR26A)
- net A4: now also J3.6 (Pin_6); no longer J3.4 (Pin_4)
- net A5: now also J3.7 (Pin_7); no longer J3.5 (Pin_5)
- net A6: now also J3.8 (Pin_8); no longer J3.6 (Pin_6)
- net A7: now also J3.9 (Pin_9); no longer J3.7 (Pin_7)
- net A8: now also J3.10 (Pin_10); no longer J3.8 (Pin_8)
- net ADC: now also R9.1, U25.1 (Z); no longer R9.2
- net ADC_A: no longer U25.1 (Z)
- net DIR_1: now also IC1.P12 (PR47D)
- net DIR_2: now also IC1.N14 (PR35D)
- net DIR_3: now also IC1.L15 (PR26B)
- net GND: now also J3.1 (Pin_1), J?.10 (Pin_10), J?.12 (Pin_12), J?.14 (Pin_14), J?.16 (Pin_16), J?.18 (Pin_18), J?.19 (Pin_19), J?.20 (Pin_20), J?.4 (Pin_4), J?.6 (Pin_6), J?.8 (Pin_8); no longer J3.10 (Pin_10)
- net S0_1: now also IC1.N11 (PR47B)
- net S0_2: now also IC1.M16 (PR26C)
- net S0_3: now also IC1.K13 (PR29A)
- net S1_1: now also IC1.P16 (PR35A)
- net S1_2: now also IC1.M15 (PR26D)
- net S1_3: now also IC1.L13 (PR29C)
- net S2_1: now also IC1.P14 (PR38B)
- net S2_2: now also IC1.M13 (PR35C)
- net S2_3: now also IC1.M14 (PR32D)
- net VCC: no longer U4.5 (VCC)
- net VCCA: now also J3.2 (Pin_2); no longer J3.9 (Pin_9)
- net VCCB: now also J?.1 (Pin_1), J?.2 (Pin_2)
- net B1_P: now reaches IC1.F1 (PL14A)
- net B2_P: now reaches IC1.H2 (PL20B)
- net at U4.3 (B0): now also R9.2; no longer R9.1
- net ADC_pull renamed pull_sel
- net ADC_sel renamed div_sel
- net B1 renamed B1_N
- net B3 renamed B3_N
- net B4 renamed B3_P
- net B5 renamed B4_N
- net B6 renamed B4_P
- net B7: no longer names the net of IC1.K2 (PL23D)
- net B8: no longer names the net of IC1.K1 (PL23C)
- net EN_pull renamed pull_en
- net pull_en: now also R45.2; no longer R45.1
- new net Sheet5D737161/target: J?.3 (Pin_3)
- new net sheet5D96E709/target: J?.5 (Pin_5)
- new net sheet5D9A1BD9/target: J?.7 (Pin_7)
- new net sheet5D9A1BDA/target: J?.9 (Pin_9)
- new net sheet5D9D50B4/target: J?.11 (Pin_11)
- new net sheet5D9D50B5/target: J?.13 (Pin_13)
- new net sheet5D9D50B6/target: J?.15 (Pin_15)
- new net sheet5D9D50B7/target: J?.17 (Pin_17)
Other:
- note added: "ADC voltage divider / pull-up / pull-down"
- note removed: "ADC pull up/down"
- note removed: "ADC voltage divider"
- note removed: "add ext clipper?"
- moved on the sheet: R18, R19, R45, R7, R9, U25, U4

Commit message: Completed routing of new connectors.
Parts:
- added U8: AT25xxx, gsg-modules:SOIC8-154, symbol Memory_EEPROM:AT25xxx
- J6: Note (none) -> DNP
- gave numbers to parts that had none: 1
Connections:
- net A1: now also J3.9 (Pin_9); no longer J3.3 (Pin_3)
- net A2: now also J3.10 (Pin_10); no longer J3.4 (Pin_4)
- net A3: now also J3.7 (Pin_7); no longer J3.5 (Pin_5)
- net A4: now also J3.8 (Pin_8); no longer J3.6 (Pin_6)
- net A5: now also J3.5 (Pin_5); no longer J3.7 (Pin_7)
- net A6: now also J3.6 (Pin_6); no longer J3.8 (Pin_8)
- net A7: now also J3.4 (Pin_4); no longer J3.9 (Pin_9)
- net A8: now also J3.3 (Pin_3); no longer J3.10 (Pin_10)
- net B2_N: now also IC1.H2 (PL20B)
- net B2_P: no longer IC1.H2 (PL20B)
- net CSSPIN: now also U8.1 (~CS)
- net GND: now also U8.4 (GND)
- net MISO: now also U8.2 (MISO)
- net MOSI: now also U8.5 (MOSI)
- net SCK: now also U8.6 (SCK)
- net VCC: now also U8.3 (~WP), U8.7 (~HOLD), U8.8 (VCC)
Other:
- note added: "SSPI: CFG[2:0] = [001] (default)\nMSPI: CFG[2:0] = [010]"
- note added: "optional SPI flash"
- note removed: "check ordering of CFG pins\nfor default setup\nSSPI: CFG[2:0] = 001"
Changed lines of the file:
@@
 $Descr USLedger 17000 11000
 encoding utf-8
-Sheet 1 10
+Sheet 1 17
 Title "GreatFET Neighbor Template"
 Date "2019-03-01"
@@
 Text Label 15850 2500 0    50   ~ 0
 VCCA
-Text Label 15350 2600 2    50   ~ 0
+Text Label 15350 2900 2    50   ~ 0
 A1
-Text Label 15850 2600 0    50   ~ 0
+Text Label 15850 2900 0    50   ~ 0
 A2
-Text Label 15350 2700 2    50   ~ 0
+Text Label 15350 2800 2    50   ~ 0
 A3
-Text Label 15850 2700 0    50   ~ 0
+Text Label 15850 2800 0    50   ~ 0
 A4
-Text Label 15350 2800 2    50   ~ 0
+Text Label 15350 2700 2    50   ~ 0
 A5
-Text Label 15850 2800 0    50   ~ 0
+Text Label 15850 2700 0    50   ~ 0
 A6
-Text Label 15350 2900 2    50   ~ 0
+Text Label 15850 2600 0    50   ~ 0
 A7
-Text Label 15850 2900 0    50   ~ 0
+Text Label 15350 2600 2    50   ~ 0
 A8
 Text Label 17700 200  2    50   ~ 0
@@
 F 2 "Connector_PinHeader_1.00mm:PinHeader_2x03_P1.00mm_Vertical_SMD" H -9750 8600 50  0001 C CNN
 F 3 "~" H -9750 8600 50  0001 C CNN
+F 4 "DNP" H -9500 8400 50  0000 C CNN "Note"
 	1    -9750 8600
 	1    0    0    -1
@@
 U 1 1 5CF0406A
 P -8250 6750
-F 0 "R58" V -8043 6750 50  0000 C CNN
-F 1 "1k" V -8134 6750 50  0000 C CNN
+F 0 "R58" V -8150 6750 50  0000 C CNN
+F 1 "1k" V -8250 6750 50  0000 C CNN
 F 2 "gsg-modules:0402" V -8320 6750 50  0001 C CNN
 F 3 "~" H -8250 6750 50  0001 C CNN
@@
 U 1 1 5CF8052D
 P -8150 7300
-F 0 "R59" V -7943 7300 50  0000 C CNN
-F 1 "4.7k" V -8034 7300 50  0000 C CNN
+F 0 "R59" V -8050 7300 50  0000 C CNN
+F 1 "4.7k" V -8150 7300 50  0000 C CNN
 F 2 "gsg-modules:0402" V -8220 7300 50  0001 C CNN
 F 3 "~" H -8150 7300 50  0001 C CNN
@@
 Text Label -8350 6200 3    50   ~ 0
 CFG_0
-Text Notes -8850 8000 0    50   ~ 0
-check ordering of CFG pins\nfor default setup\nSSPI: CFG[2:0] = 001
+Text Notes -8700 8000 0    50   ~ 0
+SSPI: CFG[2:0] = [001] (default)\nMSPI: CFG[2:0] = [010]
 $Comp
 L Device:R R57
 U 1 1 5D071140
 P -8500 7300
-F 0 "R57" V -8293 7300 50  0000 C CNN
-F 1 "4.7k" V -8384 7300 50  0000 C CNN
+F 0 "R57" V -8400 7300 50  0000 C CNN
+F 1 "4.7k" V -8500 7300 50  0000 C CNN
 F 2 "gsg-modules:0402" V -8570 7300 50  0001 C CNN
 F 3 "~" H -8500 7300 50  0001 C CNN
@@
 B2_P
 Text Label -12350 4700 1    50   ~ 0
-B2_P
+B2_N
 Wire Wire Line
 	15300 2500 15350 2500
 $Comp
-L Connector_Generic:Conn_02x10_Odd_Even J?
+L Connector_Generic:Conn_02x10_Odd_Even J4
 U 1 1 5D4FD960
 P 19350 1450
-F 0 "J?" H 19400 2067 50  0000 C CNN
+F 0 "J4" H 19400 2067 50  0000 C CNN
 F 1 "Conn_02x10_Odd_Even" H 19400 1976 50  0000 C CNN
 F 2 "Connector_PinHeader_2.54mm:PinHeader_2x10_P2.54mm_Vertical" H 19350 1450 50  0001 C CNN
@@
 P 19700 1550
 AR Path="/5C7E37E4/5D4FE67E" Ref="#PWR?"  Part="1"
-AR Path="/5D4FE67E" Ref="#PWR?"  Part="1"
-F 0 "#PWR?" H 19700 1300 50  0001 C CNN
+AR Path="/5D4FE67E" Ref="#PWR0112"  Part="1"
+F 0 "#PWR0112" H 19700 1300 50  0001 C CNN
 F 1 "GND" V 19705 1422 50  0000 R CNN
 F 2 "" H 19700 1550 50  0001 C CNN
@@
 P 19100 1950
 AR Path="/5C7E37E4/5D5989DD" Ref="#PWR?"  Part="1"
-AR Path="/5D5989DD" Ref="#PWR?"  Part="1"
-F 0 "#PWR?" H 19100 1700 50  0001 C CNN
+AR Path="/5D5989DD" Ref="#PWR0115"  Part="1"
+F 0 "#PWR0115" H 19100 1700 50  0001 C CNN
 F 1 "GND" V 19105 1822 50  0000 R CNN
 F 2 "" H 19100 1950 50  0001 C CNN
@@
 Wire Wire Line
 	18700 1650 19150 1650
+$Comp
+L Memory_EEPROM:AT25xxx U8
+U 1 1 5D0F2A29
+P -9700 9600
+F 0 "U8" H -9850 9350 50  0000 C CNN
+F 1 "AT25xxx" H -9850 9250 50  0000 C CNN
+F 2 "gsg-modules:SOIC8-154" H -9700 9600 50  0001 C CNN
+F 3 "http://ww1.microchip.com/downloads/en/DeviceDoc/Atmel-8707-SEEPROM-AT25010B-020B-040B-Datasheet.pdf" H -9700 9600 50  0001 C CNN
+F 4 "DNP" H -9900 9850 50  0000 C CNN "Note"
+	1    -9700 9600
+	1    0    0    -1
+$EndComp
+Wire Wire Line
+	-9700 9300 -9650 9300
+Wire Wire Line
+	-9700 9900 -9650 9900
+$Comp
+L power:GND #PWR0118
+U 1 1 5D161379
+P -9650 9900
+F 0 "#PWR0118" H -9650 9650 50  0001 C CNN
+F 1 "GND" V -9645 9772 50  0000 R CNN
+F 2 "" H -9650 9900 50  0001 C CNN
+F 3 "" H -9650 9900 50  0001 C CNN
+	1    -9650 9900
+	0    -1   -1   0
+$EndComp
+$Comp
+L power:VCC #PWR0119
+U 1 1 5D161602
+P -9650 9300
+F 0 "#PWR0119" H -9650 9150 50  0001 C CNN
+F 1 "VCC" V -9633 9428 50  0000 L CNN
+F 2 "" H -9650 9300 50  0001 C CNN
+F 3 "" H -9650 9300 50  0001 C CNN
+	1    -9650 9300
+	0    1    1    0
+$EndComp
+Text Notes -10000 10100 0    50   ~ 0
+optional SPI flash
+Text Label -9300 9500 0    50   ~ 0
+SCK
+Text Label -10100 9700 2    50   ~ 0
+CSSPIN
+Text Label -9300 9600 0    50   ~ 0
+MOSI
+Text Label -9300 9700 0    50   ~ 0
+MISO
+$Comp
+L power:VCC #PWR0120
+U 1 1 5D16C39C
+P -10150 9550
+F 0 "#PWR0120" H -10150 9400 50  0001 C CNN
+F 1 "VCC" V -10132 9677 50  0000 L CNN
+F 2 "" H -10150 9550 50  0001 C CNN
+F 3 "" H -10150 9550 50  0001 C CNN
+	1    -10150 9550
+	0    -1   -1   0
+$EndComp
+Wire Wire Line
+	-10150 9500 -10100 9500
+Wire Wire Line
+	-10100 9600 -10150 9600
+Wire Wire Line
+	-10150 9600 -10150 9550
+Connection ~ -10150 9550
+Wire Wire Line
+	-10150 9550 -10150 9500
 Wire Bus Line
 	-5400 2700 -3400 2700

Commit message: Completed Bank A mux routing.
Connections:
- net +5V: no longer R15.1
- net A1_shift: now also IC1.K16 (PR23C); no longer IC1.P13 (PR41A)
- net A2_shift: now also IC1.J14 (PR20C); no longer IC1.N16 (PR32A)
- net A3_shift: now also IC1.K13 (PR29A); no longer IC1.L16 (PR26A)
- net A4_shift: now also IC1.G13 (PR11B)
- net A5_shift: now also IC1.F15 (PR11C)
- net A6_shift: now also IC1.E13 (PT62B)
- net A7_shift: now also IC1.P13 (PR41A)
- net A8_shift: now also IC1.N16 (PR32A)
- net DIR_1: now also IC1.L14 (PR32C); no longer IC1.P12 (PR47D)
- net DIR_2: now also IC1.J13 (PR17C); no longer IC1.N14 (PR35D)
- net DIR_4: now also IC1.H14 (PR14D)
- net DIR_5: now also IC1.F14 (PR5D)
- net DIR_6: now also IC1.E14 (PR5C)
- net DIR_7: now also IC1.P12 (PR47D)
- net DIR_8: now also IC1.N14 (PR35D)
- net S0_1: now also IC1.K14 (PR20D); no longer IC1.N11 (PR47B)
- net S0_2: now also IC1.G16 (PR20A); no longer IC1.M16 (PR26C)
- net S0_3: now also IC1.L16 (PR26A); no longer IC1.K13 (PR29A)
- net S0_4: now also IC1.G14 (PR14C)
- net S0_5: now also IC1.C15 (PR5B)
- net S0_6: now also IC1.D16 (PR8A)
- net S0_7: now also IC1.P14 (PR38B)
- net S0_8: now also IC1.M13 (PR35C)
- net S1_1: now also IC1.K15 (PR23D); no longer IC1.P16 (PR35A)
- net S1_2: now also IC1.H15 (PR20B); no longer IC1.M15 (PR26D)
- net S1_3: now also IC1.M14 (PR32D); no longer IC1.L13 (PR29C)
- net S1_4: now also IC1.G15 (PR14B)
- net S1_5: now also IC1.D12 (PT58A)
- net S1_6: now also IC1.E15 (PR8B)
- net S1_7: now also IC1.P16 (PR35A)
- net S1_8: now also IC1.M15 (PR26D)
- net S2_1: now also IC1.J16 (PR23A); no longer IC1.P14 (PR38B)
- net S2_2: now also IC1.J15 (PR23B); no longer IC1.M13 (PR35C)
- net S2_3: now also IC1.L13 (PR29C); no longer IC1.M14 (PR32D)
- net S2_4: now also IC1.F16 (PR14A)
- net S2_5: now also IC1.E12 (PT58B)
- net S2_6: now also IC1.E16 (PR11D)
- net S2_7: now also IC1.N11 (PR47B)
- net S2_8: now also IC1.M16 (PR26C)
- net VCC: now also R15.1
- net J2.38: no longer names the net of J2.38 (Pin_38)
- net J2.38: no longer IC1.C15 (PR5B)
- net div_sel renamed div_en
- no-connect marks 0 -> 1
Changed lines of the file:
@@
 Text Label -3700 3000 1    50   ~ 0
 J2.36
-Text Label -3600 3000 1    50   ~ 0
-J2.38
 Text Label -3500 3000 1    50   ~ 0
 J2.40
@@
 $EndComp
 $Comp
-L power:+5V #PWR?
-U 1 1 5D7BE9FA
-P 11900 6550
-AR Path="/5C842523/5D7BE9FA" Ref="#PWR?"  Part="1"
-AR Path="/5D7BE9FA" Ref="#PWR0133"  Part="1"
-F 0 "#PWR0133" H 11900 6400 50  0001 C CNN
-F 1 "+5V" V 11915 6678 50  0000 L CNN
-F 2 "" H 11900 6550 50  0001 C CNN
-F 3 "" H 11900 6550 50  0001 C CNN
-	1    11900 6550
-	1    0    0    -1
-$EndComp
-$Comp
 L power:GND #PWR?
 U 1 1 5D7BEA01
@@
 Text Label 11900 7000 0    50   ~ 0
 SSEL
-Wire Wire Line
-	11900 6550 11900 6600
 $Comp
 L Device:C C13
@@
 Connection ~ 11600 7200
 Text Label 11950 3100 2    50   ~ 0
-div_sel
+div_en
 $Comp
 L gsg-symbols:LFE5U-12F-6BG256C IC1
@@
 Text Label -5750 4700 1    50   ~ 0
 J2.40
-Text Label -5650 4700 1    50   ~ 0
-J2.38
 Text Label -5550 4700 1    50   ~ 0
 J2.36
@@
 	14100 6600 14400 6600
 Text Label -10150 6200 3    50   ~ 0
-DIR_1
+DIR_7
 Text Label -10250 6200 3    50   ~ 0
-A1_shift
+A7_shift
 Text Label -10350 6200 3    50   ~ 0
-S2_1
+S0_7
 Text Label -10550 6200 3    50   ~ 0
-S1_1
+S1_7
 Text Label -8450 6200 3    50   ~ 0
-S0_1
+S2_7
 Text Label -8750 6200 3    50   ~ 0
-DIR_2
+DIR_8
 Text Label -8950 6200 3    50   ~ 0
-A2_shift
+A8_shift
 Text Label -7050 6200 3    50   ~ 0
-S2_2
+S0_8
 Text Label -7250 6200 3    50   ~ 0
-S1_2
+S1_8
 Text Label -7350 6200 3    50   ~ 0
-S0_2
+S2_8
 Text Label -5650 6200 3    50   ~ 0
 DIR_3
 Text Label -5750 6200 3    50   ~ 0
-A3_shift
+S0_3
 Text Label -7150 6200 3    50   ~ 0
-S2_3
-Text Label -5450 6200 3    50   ~ 0
 S1_3
+Text Label -5450 6200 3    50   ~ 0
+S2_3
 Text Label -3850 6200 3    50   ~ 0
-S0_3
+A3_shift
 Wire Wire Line
 	12650 2900 12700 2900
@@
 Wire Wire Line
 	-10150 9550 -10150 9500
+Text Label -5550 6200 3    50   ~ 0
+DIR_1
+Text Label -4150 6200 3    50   ~ 0
+A1_shift
+Text Label -3950 6200 3    50   ~ 0
+S0_1
+Text Label -4050 6200 3    50   ~ 0
+S1_1
+Text Label -2550 6200 3    50   ~ 0
+S2_1
+Text Label -2450 6200 3    50   ~ 0
+S2_2
+Text Label -13650 4700 1    50   ~ 0
+S1_2
+Text Label -2250 6200 3    50   ~ 0
+DIR_2
+Text Label -2350 6200 3    50   ~ 0
+A2_shift
+Text Label -12150 4700 1    50   ~ 0
+S0_2
+Text Label -13550 4700 1    50   ~ 0
+DIR_4
+Text Label -11850 4700 1    50   ~ 0
+A4_shift
+Text Label -11950 4700 1    50   ~ 0
+S0_4
+Text Label -12050 4700 1    50   ~ 0
+S1_4
+Text Label -10550 4700 1    50   ~ 0
+S2_4
+Text Label -7350 4700 1    50   ~ 0
+S0_6
+Text Label -8850 4700 1    50   ~ 0
+S1_6
+Text Label -8950 4700 1    50   ~ 0
+S2_6
+Text Label -8650 4700 1    50   ~ 0
+A6_shift
+Text Label -8750 4700 1    50   ~ 0
+DIR_6
+Text Label -5650 4700 1    50   ~ 0
+S0_5
+Text Label -6950 4700 1    50   ~ 0
+S1_5
+Text Label -8550 4700 1    50   ~ 0
+S2_5
+Text Label -10350 4700 1    50   ~ 0
+DIR_5
+Text Label -10450 4700 1    50   ~ 0
+A5_shift
+$Comp
+L power:VCC #PWR0129
+U 1 1 5D150A98
+P 11900 6300
+F 0 "#PWR0129" H 11900 6150 50  0001 C CNN
+F 1 "VCC" H 11917 6473 50  0000 C CNN
+F 2 "" H 11900 6300 50  0001 C CNN
+F 3 "" H 11900 6300 50  0001 C CNN
+	1    11900 6300
+	1    0    0    -1
+$EndComp
+Wire Wire Line
+	11900 6300 11900 6600
+NoConn ~ -3600 3000
 Wire Bus Line
 	-5400 2700 -3400 2700

Commit message: Added I2C IO expander
Parts:
- added R71, R72: 10k, gsg-modules:0402, symbol Device:R
- added U26: PCA6408A, gsg-modules:TSSOP16, symbol gsg-symbols:PCA6408A
Connections:
- net +5V: now also R15.1, U26.16 (VDD(P)), U26.2 (ADDR)
- net COUT1: now also U26.9 (P4)
- net COUT2: now also U26.10 (P5)
- net DAC2_EN: now also U26.4 (P0)
- net GND: now also U26.8 (VSS)
- net J2.39: now also U26.15 (SDA)
- net J2.40: now also U26.14 (SCL)
- net SSEL: no longer R15.2, U7.9 (~SYNC~)
- net VCC: now also R71.2, R72.1, U26.1 (VDD); no longer R15.1
- net VCCA_EN: now also U26.12 (P7)
- net VCCB_EN: now also U26.11 (P6)
- net div_en: now also IC1.M3 (PL32D)
- net pull_en: now also IC1.P3 (PL38B)
- net pull_sel: now also IC1.P4 (PL41A)
- new net: R72.2, U26.13 (~INT~)
- new net: R71.1, U26.3 (~RESET~)
- new net DAC~SYNC~: R15.2, U26.7 (P3), U7.9 (~SYNC~)
- no-connect marks 1 -> 3
Other:
- note added: "also comes in smaller/cheaper packages"
Changed lines of the file:
@@
 MOSI
 Text Label 11900 7000 0    50   ~ 0
-SSEL
+DAC~SYNC~
 $Comp
 L Device:C C13
@@
 Text Label -10450 4700 1    50   ~ 0
 A5_shift
+Wire Wire Line
+	11900 6300 11900 6600
+NoConn ~ -3600 3000
+Text Label -9350 6200 3    50   ~ 0
+pull_sel
+Text Label -9250 6200 3    50   ~ 0
+pull_en
+Text Label -6050 6200 3    50   ~ 0
+div_en
 $Comp
-L power:VCC #PWR0129
-U 1 1 5D150A98
+L gsg-symbols:PCA6408A U26
+U 1 1 5D21CE35
+P 11150 8600
+F 0 "U26" H 11050 9075 50  0000 C CNN
+F 1 "PCA6408A" H 11050 8984 50  0000 C CNN
+F 2 "gsg-modules:TSSOP16" H 11150 8600 50  0001 C CNN
+F 3 "" H 11150 8600 50  0001 C CNN
+F 4 "NXP USA Inc." H 11150 8600 50  0001 C CNN "Manufacturer"
+F 5 "PCA6408APW,118" H 11150 8600 50  0001 C CNN "Part Number"
+F 6 "IC I/O EXPANDER 8BIT GP 16TSSOP" H 11150 8600 50  0001 C CNN "Description"
+	1    11150 8600
+	1    0    0    -1
+$EndComp
+Text Label 11400 8550 0    50   ~ 0
+J2.40
+Text Label 11400 8450 0    50   ~ 0
+J2.39
+$Comp
+L power:+5V #PWR?
+U 1 1 5D2210DF
 P 11900 6300
+AR Path="/5C842523/5D2210DF" Ref="#PWR?"  Part="1"
+AR Path="/5D2210DF" Ref="#PWR0129"  Part="1"
 F 0 "#PWR0129" H 11900 6150 50  0001 C CNN
-F 1 "VCC" H 11917 6473 50  0000 C CNN
+F 1 "+5V" V 11915 6428 50  0000 L CNN
 F 2 "" H 11900 6300 50  0001 C CNN
 F 3 "" H 11900 6300 50  0001 C CNN
@@
 	1    0    0    -1
 $EndComp
+$Comp
+L power:+5V #PWR?
+U 1 1 5D221375
+P 11450 8350
+AR Path="/5C842523/5D221375" Ref="#PWR?"  Part="1"
+AR Path="/5D221375" Ref="#PWR0130"  Part="1"
+F 0 "#PWR0130" H 11450 8200 50  0001 C CNN
+F 1 "+5V" V 11465 8478 50  0000 L CNN
+F 2 "" H 11450 8350 50  0001 C CNN
+F 3 "" H 11450 8350 50  0001 C CNN
+	1    11450 8350
+	0    1    1    0
+$EndComp
 Wire Wire Line
-	11900 6300 11900 6600
-NoConn ~ -3600 3000
+	11400 8350 11450 8350
+$Comp
+L power:+5V #PWR?
+U 1 1 5D25A151
+P 10650 8450
+AR Path="/5C842523/5D25A151" Ref="#PWR?"  Part="1"
+AR Path="/5D25A151" Ref="#PWR0131"  Part="1"
+F 0 "#PWR0131" H 10650 8300 50  0001 C CNN
+F 1 "+5V" V 10665 8578 50  0000 L CNN
+F 2 "" H 10650 8450 50  0001 C CNN
+F 3 "" H 10650 8450 50  0001 C CNN
+	1    10650 8450
+	0    -1   -1   0
+$EndComp
+Wire Wire Line
+	10700 8450 10650 8450
+$Comp
+L power:VCC #PWR0133
+U 1 1 5D29349A
+P 10650 8350
+F 0 "#PWR0133" H 10650 8200 50  0001 C CNN
+F 1 "VCC" V 10650 8550 50  0000 C CNN
+F 2 "" H 10650 8350 50  0001 C CNN
+F 3 "" H 10650 8350 50  0001 C CNN
+	1    10650 8350
+	0    -1   -1   0
+$EndComp
+Wire Wire Line
+	10650 8350 10700 8350
+$Comp
+L Device:R R?
+U 1 1 5D2CDC23
+P 10250 8550
+AR Path="/5C7E37E4/5D2CDC23" Ref="R?"  Part="1"
+AR Path="/5D2CDC23" Ref="R71"  Part="1"
+F 0 "R71" H 10180 8504 50  0000 R CNN
+F 1 "10k" V 10250 8600 50  0000 R CNN
+F 2 "gsg-modules:0402" V 10180 8550 50  0001 C CNN
+F 3 "~" H 10250 8550 50  0001 C CNN
+	1    10250 8550
+	0    1    1    0
+$EndComp
+Wire Wire Line
+	10700 8550 10400 8550
+$Comp
+L power:VCC #PWR0137
+U 1 1 5D307922
+P 10100 8550
+F 0 "#PWR0137" H 10100 8400 50  0001 C CNN
+F 1 "VCC" V 10100 8750 50  0000 C CNN
+F 2 "" H 10100 8550 50  0001 C CNN
+F 3 "" H 10100 8550 50  0001 C CNN
+	1    10100 8550
+	0    -1   -1   0
+$EndComp
+$Comp
+L power:GND #PWR0138
+U 1 1 5D308848
+P 10650 9050
+F 0 "#PWR0138" H 10650 8800 50  0001 C CNN
+F 1 "GND" V 10655 8922 50  0000 R CNN
+F 2 "" H 10650 9050 50  0001 C CNN
+F 3 "" H 10650 9050 50  0001 C CNN
+	1    10650 9050
+	0    1    1    0
+$EndComp
+Wire Wire Line
+	10650 9050 10700 9050
+$Comp
+L Device:R R?
+U 1 1 5D3425EF
+P 11850 8650
+AR Path="/5C7E37E4/5D3425EF" Ref="R?"  Part="1"
+AR Path="/5D3425EF" Ref="R72"  Part="1"
+F 0 "R72" H 11780 8604 50  0000 R CNN
+F 1 "10k" V 11850 8700 50  0000 R CNN
+F 2 "gsg-modules:0402" V 11780 8650 50  0001 C CNN
+F 3 "~" H 11850 8650 50  0001 C CNN
+	1    11850 8650
+	0    1    1    0
+$EndComp
+$Comp
+L power:VCC #PWR0139
+U 1 1 5D37C3BC
+P 12050 8650
+F 0 "#PWR0139" H 12050 8500 50  0001 C CNN
+F 1 "VCC" V 12050 8850 50  0000 C CNN
+F 2 "" H 12050 8650 50  0001 C CNN
+F 3 "" H 12050 8650 50  0001 C CNN
+	1    12050 8650
+	0    1    1    0
+$EndComp
+Wire Wire Line
+	12000 8650 12050 8650
+Text Label 10700 8950 2    50   ~ 0
+DAC~SYNC~
+Text Label 11400 8750 0    50   ~ 0
+VCCA_EN
+Text Label 10700 8650 2    50   ~ 0
+DAC2_EN
+Text Label 11400 8850 0    50   ~ 0
+VCCB_EN
+Text Label 11400 9050 0    50   ~ 0
+COUT1
+Text Label 11400 8950 0    50   ~ 0
+COUT2
+Text Notes 10300 9200 0    50   ~ 0
+also comes in smaller/cheaper packages
+NoConn ~ 10700 8750
+NoConn ~ 10700 8850
+Wire Wire Line
+	11400 8650 11700 8650
 Wire Bus Line
 	-5400 2700 -3400 2700

Commit message: Completed routing
Connections:
- net VCCIO0 is gone; now on net VCC: IC1.F6 (VCCIO0_1), IC1.F7 (VCCIO0_2)
- net div_en: now also U26.6 (P2); no longer IC1.M3 (PL32D)
- net J2.38: now reaches J2.38 (Pin_38)
- net J2.38: now also IC1.M3 (PL32D)
- no-connect marks 3 -> 1
Changed lines of the file:
@@
 Wire Wire Line
 	-13250 4700 -13250 4650
-Text Label -11100 1150 2    50   ~ 0
+Text Label -11000 1150 2    50   ~ 0
 VCCIO1
 $Comp
@@
 Wire Wire Line
 	11900 6300 11900 6600
-NoConn ~ -3600 3000
 Text Label -9350 6200 3    50   ~ 0
 pull_sel
@@
 pull_en
 Text Label -6050 6200 3    50   ~ 0
-div_en
+J2.38
 $Comp
 L gsg-symbols:PCA6408A U26
@@
 also comes in smaller/cheaper packages
 NoConn ~ 10700 8750
-NoConn ~ 10700 8850
 Wire Wire Line
 	11400 8650 11700 8650
@@
 Wire Bus Line
 	-2150 4150 -400 4150
+Text Label 10700 8850 2    50   ~ 0
+div_en
+Text Label -3600 3000 1    50   ~ 0
+J2.38
+Text Label -11350 1150 2    50   ~ 0
+VCCIO0
 $EndSCHEMATC

Commit message: Matched path length of bank B differential pairs
Connections:
- net VCCB: no longer J4.2 (Pin_2)
- net Sheet5D737161/target renamed B1T_P
- net sheet5D96E709/target renamed B1T_N
- net sheet5D9A1BD9/target renamed B2T_P
- net sheet5D9A1BDA/target renamed B2T_N
- net sheet5D9D50B4/target renamed B3T_P
- net sheet5D9D50B5/target renamed B3T_N
- net sheet5D9D50B6/target renamed B4T_P
- net sheet5D9D50B7/target renamed B4T_N
- new net Vtarget: J4.2 (Pin_2)
Other:
- note added: "to ADC? DNP?"
Changed lines of the file:
@@
 Text Label 19150 1050 2    50   ~ 0
-VCCB
-Text Label 19650 1050 0    50   ~ 0
 VCCB
 $Comp
@@
 Wire Wire Line
 	11400 8650 11700 8650
+Text Label 10700 8850 2    50   ~ 0
+div_en
+Text Label -3600 3000 1    50   ~ 0
+J2.38
+Text Label -11350 1150 2    50   ~ 0
+VCCIO0
 Wire Bus Line
 	-5400 2700 -3400 2700
@@
 Wire Bus Line
 	-2150 4150 -400 4150
-Text Label 10700 8850 2    50   ~ 0
-div_en
-Text Label -3600 3000 1    50   ~ 0
-J2.38
-Text Label -11350 1150 2    50   ~ 0
-VCCIO0
+Text Label 18800 200  2    50   ~ 0
+B1T_P
+Text Label 18800 550  2    50   ~ 0
+B1T_N
+Text Label 18750 900  2    50   ~ 0
+B2T_P
+Text Label 18700 1250 2    50   ~ 0
+B2T_N
+Text Label 18700 1600 2    50   ~ 0
+B3T_P
+Text Label 18600 1950 2    50   ~ 0
+B3T_N
+Text Label 18600 2300 2    50   ~ 0
+B4T_P
+Text Label 18600 2650 2    50   ~ 0
+B4T_N
+Text Label 19650 1050 0    50   ~ 0
+Vtarget
+Text Notes 19950 1050 0    50   ~ 0
+to ADC? DNP?
 $EndSCHEMATC
