File: foxglove.sch (KiCad schematic (older format))
At the start: 95 parts, among them IC1 LFE5U-12F-6BG256C, J1 NEIGHBOR1, J2 NEIGHBOR2, J3 Conn_02x05_Odd_Even, J4 Conn_02x10_Odd_Even, J5 Conn_01x02_Female, J6 Conn_02x03_Odd_Even, J7 BONUS_ROW, U1 LM393, U2 ADP225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

Commit message: Changed bank A footprint and rearranged silkscreen
Parts:
- added R73: 0, gsg-modules:0402, symbol Device:R
- J3: footprint gsg-modules:2X5-SHROUDED -> Connector_PinHeader_2.54mm:PinHeader_2x05_P2.54mm_Vertical; Description Conn Shrouded Header F 10 POS 2.54mm Solder ST Thru-Hole -> CONN HEADER R/A 10POS 2.54MM; Manufacturer SparkFun Electronics -> Sullins Connector Solutions; Part Number PRT-08506 -> SBH11-PBPC-D05-RA-BK
- J4: Description (none) -> CONN HEADER R/A 20POS 2.54MM; Manufacturer (none) -> Sullins Connector Solutions; Part Number (none) -> SBH11-PBPC-D10-RA-BK
Connections:
- net ADC_A: now also R73.1
- net Vtarget: now also R73.2
Other:
- note removed: "to ADC? DNP?"
Changed lines of the file:
@@
 F 0 "J3" H 15600 3117 50  0000 C CNN
 F 1 "Conn_02x05_Odd_Even" H 15600 3026 50  0000 C CNN
-F 2 "gsg-modules:2X5-SHROUDED" H 15550 2700 50  0001 C CNN
+F 2 "Connector_PinHeader_2.54mm:PinHeader_2x05_P2.54mm_Vertical" H 15550 2700 50  0001 C CNN
 F 3 "~" H 15550 2700 50  0001 C CNN
-F 4 "SparkFun Electronics" H 15550 2700 50  0001 C CNN "Manufacturer"
-F 5 "PRT-08506" H 15550 2700 50  0001 C CNN "Part Number"
-F 6 "Conn Shrouded Header F 10 POS 2.54mm Solder ST Thru-Hole" H 15550 2700 50  0001 C CNN "Description"
+F 4 "Sullins Connector Solutions" H 15550 2700 50  0001 C CNN "Manufacturer"
+F 5 "SBH11-PBPC-D05-RA-BK" H 15550 2700 50  0001 C CNN "Part Number"
+F 6 "CONN HEADER R/A 10POS 2.54MM" H 15550 2700 50  0001 C CNN "Description"
 	1    15550 2700
 	1    0    0    -1
@@
 F 2 "Connector_PinHeader_2.54mm:PinHeader_2x10_P2.54mm_Vertical" H 19350 1450 50  0001 C CNN
 F 3 "~" H 19350 1450 50  0001 C CNN
+F 4 "Sullins Connector Solutions" H 19350 1450 50  0001 C CNN "Manufacturer"
+F 5 "SBH11-PBPC-D10-RA-BK" H 19350 1450 50  0001 C CNN "Part Number"
+F 6 "CONN HEADER R/A 20POS 2.54MM" H 19350 1450 50  0001 C CNN "Description"
 	1    19350 1450
 	1    0    0    -1
@@
 Text Label -11350 1150 2    50   ~ 0
 VCCIO0
-Wire Bus Line
-	-5400 2700 -3400 2700
-Wire Bus Line
-	-5700 3800 -3400 3800
-Wire Bus Line
-	-13800 8000 -10900 8000
-Wire Bus Line
-	-12700 9100 -10900 9100
-Wire Bus Line
-	-2150 4150 -400 4150
 Text Label 18800 200  2    50   ~ 0
 B1T_P
@@
 Text Label 19650 1050 0    50   ~ 0
 Vtarget
-Text Notes 19950 1050 0    50   ~ 0
-to ADC? DNP?
+Wire Wire Line
+	19650 1050 19950 1050
+Wire Bus Line
+	-5400 2700 -3400 2700
+Wire Bus Line
+	-5700 3800 -3400 3800
+Wire Bus Line
+	-13800 8000 -10900 8000
+Wire Bus Line
+	-12700 9100 -10900 9100
+Wire Bus Line
+	-2150 4150 -400 4150
+$Comp
+L Device:R R?
+U 1 1 5D235AE1
+P 20100 1050
+AR Path="/5C7E37E4/5D235AE1" Ref="R?"  Part="1"
+AR Path="/5D235AE1" Ref="R73"  Part="1"
+F 0 "R73" V 20200 1050 50  0000 C CNN
+F 1 "0" V 20100 1050 50  0000 C CNN
+F 2 "gsg-modules:0402" V 20030 1050 50  0001 C CNN
+F 3 "~" H 20100 1050 50  0001 C CNN
+F 4 "DNP" V 20000 1050 50  0000 C CNN "Note"
+	1    20100 1050
+	0    1    1    0
+$EndComp
+Text Label 20250 1050 0    50   ~ 0
+ADC_A
 $EndSCHEMATC

Commit message: Added silkscreen tables for banks and completed BOM data
Parts:
- C10, C2, C9: Description (none) -> CAP CER 4.7UF 10V X5R 0402; Manufacturer (none) -> Murata Electronics North America; Part Number (none) -> GRM155R61A475MEAAD
- C11, C12, C3: Description (none) -> CAP CER 2700PF 50V X7R 0402; Manufacturer (none) -> Yageo; Part Number (none) -> CC0402KRX7R9BB272
- C18, C19, C23, C24, C25, C29, C30, C33, C34: value 100nF -> 0.1uF
- IC1: Manufacturer (none) -> Lattice; Part Number (none) -> LFE5U-12F-6BG256C
- R1, R2, R3, R4, R5, R56, R57, R59, R6, R60: Description (none) -> RES 4.7K OHM 5% 1/16W 0402; Manufacturer (none) -> Stackpole Electronics Inc; Part Number (none) -> RMCF0402JT4K70
- R11, R13, R21: Description (none) -> RES 20K OHM 5% 1/16W 0402; Manufacturer (none) -> Stackpole Electronics Inc; Part Number (none) -> RMCF0402JT20K0
- R12: Description (none) -> RES 57.6K OHM 1% 1/16W 0402; Manufacturer (none) -> Stackpole Electronics Inc; Part Number (none) -> RMCF0402FT57K6
- R14, R16: Description (none) -> RES 118K OHM 1% 1/16W 0402; Manufacturer (none) -> Stackpole Electronics Inc; Part Number (none) -> RMCF0402FT118K
- R15, R18, R19, R45, R7, R71, R72: Description (none) -> RES 10K OHM 5% 1/16W 0402; Manufacturer (none) -> Stackpole Electronics Inc; Part Number (none) -> RMCF0402JT10K0
- R22, R8: Description (none) -> RES 88.7K OHM 1% 1/16W 0402; Manufacturer (none) -> Stackpole Electronics Inc; Part Number (none) -> RMCF0402FT88K7
- R41: Description (none) -> RES SMD 25K OHM 0.1% 1/20W 0402; Manufacturer (none) -> Vishay Dale; Part Number (none) -> PNM0402E2502BST1
- R42, R43: Description (none) -> RES 100K OHM 5% 1/16W 0402; Manufacturer (none) -> Stackpole Electronics Inc; Part Number (none) -> RMCF0402JT100K
- R44: Description (none) -> RES 120K OHM 1% 1/16W 0402; Manufacturer (none) -> Stackpole Electronics Inc; Part Number (none) -> RMCF0402FT120K
- R58: Description (none) -> RES 1K OHM 5% 1/10W 0402; Manufacturer (none) -> KOA Speer Electronics, Inc.; Part Number (none) -> RK73B1ETTP102J
- R63: Description (none) -> RES 127K OHM 1% 1/16W 0402; Manufacturer (none) -> Stackpole Electronics Inc; Part Number (none) -> RMCF0402FT127K
- R9: Description (none) -> RES SMD 5K OHM 0.1% 1/20W 0402; Manufacturer (none) -> Vishay Dale; Part Number (none) -> PNM0402E5001BST1
- U25: Description (none) -> IC MUX/DEMUX 2X1 8VSSOP; Manufacturer (none) -> Nexperia USA Inc.; Part Number (none) -> 74LVC1G53DC,125
Connections:
- net +5V: now also R45.2; no longer R45.1
- net GND: now also R18.1; no longer R18.2
- net VCCA: now also R19.1; no longer R19.2
- net pull_en: now also R45.1; no longer R45.2
- net at U25.6 (Y1): now also R19.2; no longer R19.1
- net at U25.7 (Y0): now also R18.2; no longer R18.1
